File: bay-station/bay-station.kicad_pcb (KiCad board)
At the start: 2 copper layers, 0 parts

Commit message: Give the bay station its real 4-layer stackup
bay-station.kicad_pcb was an 86-line stub: KiCad's 2-layer default, board
thickness 1.6 mm, nothing on it. That directly contradicted a decision the
docs had been carrying as settled since the architecture swap -- DW3000
Section 7.3 forces a controlled-impedance build of at least four layers,
and the file said two.

Set from DW3000 Datasheet v1.3, Section 7.3.2 Figure 35 "Recommended QFN
Stack-up". Figure 35 is the right one because this board uses DW3210
(QFN40); Figure 34 is the WLCSP variant and does not apply:

    F.Cu     35 um
    prepreg 254 um
    In1.Cu   35 um
    core    400 um
    In2.Cu   35 um
    prepreg 254 um
    B.Cu     35 um     = 1.048 mm finished

Section 7.3's remaining requirements went on the board's Cmts.User layer
rather than into another doc, because they are layout instructions and
that is where layout will see them: 50 ohm RF1/RF2 with the 2 pF DC-block
pads embedded in the track at full width, ground removed under each
DW3210 on F.Cu and In1.Cu with In2.Cu as the first solid plane, and
analog/power/digital groups kept apart.

The dielectric constants are NOT datasheet values -- Figure 35 gives
thicknesses only. KiCad's FR4 defaults (er 4.5, tan d 0.02) are in the
file as placeholders, and the note says so. Controlled impedance means
the fab's stackup governs, and 1.048 mm is not a catalogue thickness.

Also: default netclass clearance 0.2 mm -> 0.15 mm. The DW3210 cannot
satisfy 0.2 mm. KiCad's QFN-40-1EP_5x5mm_P0.4mm_EP3.6x3.6mm has 0.25 mm
pads on a 0.4 mm pitch, leaving exactly 0.15 mm between neighbours, so at
0.2 mm every adjacent pad pair on all four anchors would have failed DRC
the moment footprints were placed.

Deliberately NOT done, both worth stating:

- **No footprints imported.** Every sheet is placement-only, so
  `kicad-cli sch export netlist` returns zero nets -- an import now gives
  an unconnected pile with no ratsnest and gets redone after wiring.
  Wiring the sheets is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
Other:
- copper layers 2 -> 4
- board text added: "BAY STATION -- 4-LAYER CONTROLLED-IMPEDANCE STACKUP Set 2026-09-23 from DW3000 Datasheet v1.3, Section 7.3.2 Figure 35 (Recommended QFN Stack-up) -- the variant that applies to the DW3210 QFN40: F.Cu 35um / prepreg 254um / In1.Cu 35um / core 400um / In2.Cu 35um / prepreg 254um / B.Cu 35um = 1.048mm finished Section 7.3 also requires the following, NONE of which is done yet: - RF1/RF2 routed as 50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"
Changed lines of the file:
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@@
 	(generator_version "8.0")
 	(general
-		(thickness 1.6)
+		(thickness 1.048)
 		(legacy_teardrops no)
 	)
@@
 	(layers
 		(0 "F.Cu" signal)
+		(1 "In1.Cu" signal)
+		(2 "In2.Cu" signal)
 		(31 "B.Cu" signal)
 		(32 "B.Adhes" user "B.Adhesive")
@@
 	)
 	(setup
+		(stackup
+			(layer "F.SilkS"
+				(type "Top Silk Screen")
+			)
+			(layer "F.Paste"
+				(type "Top Solder Paste")
+			)
+			(layer "F.Mask"
+				(type "Top Solder Mask")
+				(thickness 0.01)
+			)
+			(layer "F.Cu"
+				(type "copper")
+				(thickness 0.035)
+			)
+			(layer "dielectric 1"
+				(type "prepreg")
+				(thickness 0.254)
+				(material "FR4")
+				(epsilon_r 4.5)
+				(loss_tangent 0.02)
+			)
+			(layer "In1.Cu"
+				(type "copper")
+				(thickness 0.035)
+			)
+			(layer "dielectric 2"
+				(type "core")
+				(thickness 0.4)
+				(material "FR4")
+				(epsilon_r 4.5)
+				(loss_tangent 0.02)
+			)
+			(layer "In2.Cu"
+				(type "copper")
+				(thickness 0.035)
+			)
+			(layer "dielectric 3"
+				(type "prepreg")
+				(thickness 0.254)
+				(material "FR4")
+				(epsilon_r 4.5)
+				(loss_tangent 0.02)
+			)
+			(layer "B.Cu"
+				(type "copper")
+				(thickness 0.035)
+			)
+			(layer "B.Mask"
+				(type "Bottom Solder Mask")
+				(thickness 0.01)
+			)
+			(layer "B.Paste"
+				(type "Bottom Solder Paste")
+			)
+			(layer "B.SilkS"
+				(type "Bottom Silk Screen")
+			)
+			(copper_finish "None")
+			(dielectric_constraints no)
+		)
 		(pad_to_mask_clearance 0)
 		(allow_soldermask_bridges_in_footprints no)
@@
 		)
 	)
+	(gr_text "BAY STATION -- 4-LAYER CONTROLLED-IMPEDANCE STACKUP\nSet 2026-09-23 from DW3000 Datasheet v1.3, Section 7.3.2 Figure 35\n(Recommended QFN Stack-up) -- the variant that applies to the DW3210 QFN40:\n  F.Cu 35um / prepreg 254um / In1.Cu 35um / core 400um /\n  In2.Cu 35um / prepreg 254um / B.Cu 35um  =  1.048mm finished\n\nSection 7.3 also requires the following, NONE of which is done yet:\n  - RF1/RF2 routed as 50 ohm impedance-controlled lines, with the 2pF\n    DC-block pads embedded in the track at the same width so there is\n    no discontinuity.\n  - Ground copper REMOVED under each DW3210 on F.Cu and In1.Cu. In2.Cu\n    is the first SOLID ground plane. If this stackup is ever changed,\n    that first solid plane must stay at least 0.25mm below F.Cu.\n  - Analog (RF1, RF2, XIN, XOUT), power and digital groups kept apart.\n\nMaterial is KiCad's FR4 default (er 4.5, tan d 0.02). That is NOT from\nthe datasheet, which gives thicknesses only. Controlled impedance means\nthe fab's real stackup governs -- get their numbers and re-solve trace\nwidths before trusting any 50 ohm geometry.\n\nNo board outline exists yet (Edge.Cuts is empty), which is the one open\nDRC violation, and no footprints are placed. See bay-station/README.md."
+		(at 20 20 0)
+		(layer "Cmts.User")
+		(effects
+			(font
+				(size 1.5 1.5)
+				(thickness 0.25)
+			)
+			(justify left top)
+		)
+	)
