File: bay-station/connectivity.kicad_sch (KiCad schematic)
At the start: 4 parts, among them U3 BT840

Commit message: Add the missing I2C pull-ups; audit the design for level shifters
R37 (SDA), R38 (SCL), R39 (MAX17048 ALRT), all 2.2k to +3V3, on
connectivity.kicad_sch. The bay station had ZERO I2C pull-ups while
carrying three devices on the bus: MAX17048 (0x36), LIS3MDL (0x1C/0x1E),
LIS2DH (0x18/0x19). I2C is open-drain and cannot return to a logic high
without them, so this was a functional gap, not a refinement.

power_bms_notes.md had already flagged this and deliberately deferred it,
because the right pull-up rail is the host's logic supply and the host was
then an unbuilt ESP32-S3. That reasoning was correct; the host is now the
3.3 V BT840, so it is decidable. The pull-ups live on the host's sheet, not
on power_bms.

2.2k is derived, not defaulted:
- Lower bound Rp(min) = (3.3-0.4)/4mA = 725 ohm, from the strongest sink on
  the bus (MAX17048 19-6171 Rev 7: VOL 0.4 V at IOL 4 mA). 2.2k sinks
  1.32 mA.
- Upper bound from the I2C-bus spec (NXP UM10204, tr = 0.8473*Rp*Cb): 2.2k
  allows 161 pF of bus capacitance at 400 kHz against only 75 pF for a
  default 4.7k. This bus runs from power_bms to gnss across the board, so
  75 pF is too tight to assume.

LEVEL SHIFTER AUDIT: none are needed anywhere, on either board, provided
the I2C bus is pulled to +3V3 and never to VBATT_PROT.

Everything digital is 3.3 V-native: DW3210 (VDD1 1.62-3.6 V and it supplies
the I/O), BT840/nRF52840 (1.7-3.6 V), MAX-M10S (V_IO tied to VCC), LIS3MDL
and LIS2DH (separate VDD_IO), ESP32-C5 (3.0-3.6 V). The wristband has no
I2C bus at all; its 5.1k CC resistors are mandatory USB-C pull-DOWNS.

The one apparent problem is the MAX17048, whose VDD is the battery rail
because it senses cell voltage through that pin. It is not a problem, per
datasheet 19-6171 Rev 7:
- I2C is open-drain, so the bus never exceeds the pull-up rail regardless
  of any device's own supply.
- Its VIH is a FIXED 1.4 V, not 0.7*VDD, so it reads a 3.3 V bus correctly
  even at 4.2 V VDD.
- SDA/SCL/ALRT are rated -0.3 to +5.5 V abs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
Parts:
- added R37, R38, R39: 2.2k, symbol Device:R
Changed lines of the file:
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@@
+		)
+	)
+	(symbol
+		(lib_id "Device:R")
+		(at 152.4 88.9 0)
+		(unit 1)
+		(exclude_from_sim no)
+		(in_bom yes)
+		(on_board yes)
+		(dnp no)
+		(property "Reference" "R37"
+			(at 152.4 85.09 0)
+			(effects
+				(font
+					(size 1.27 1.27)
+				)
+			)
+		)
+		(property "Value" "2.2k"
+			(at 152.4 92.71 0)
+			(effects
+				(font
+					(size 1.27 1.27)
+				)
+			)
+		)
+		(property "Footprint" ""
+			(at 152.4 88.9 0)
+			(effects
+				(font
+					(size 1.27 1.27)
+				)
+				(hide yes)
+			)
+		)
+		(property "Datasheet" "~"
+			(at 152.4 88.9 0)
+			(effects
+				(font
+					(size 1.27 1.27)
+				)
+				(hide yes)
+			)
+		)
+		(property "Description" "I2C SDA pull-up for the shared housekeeping bus (MAX17048 0x36, LIS3MDL 0x1C/0x1E, LIS2DH 0x18/0x19). Value derived, not defaulted: Rp(min) = (3V3 - VOL)/IOL = (3.3-0.4)/4mA = 725 ohm from the strongest sink on the bus (MAX17048 datasheet 19-6171 Rev 7: VOL 0.4 V at IOL 4 mA). 2.2k sinks 1.32 mA, well inside that, and by the I2C-bus spec (NXP UM10204, tr = 0.8473*Rp*Cb) allows 161 pF of bus capacitance at 400 kHz versus only 75 pF for a default 4.7k -- too tight for a bus that crosses from power_bms to gnss. MUST pull up to +3V3, NEVER to VBATT_PROT: the MAX17048's VDD is the battery rail and reaches 4.2 V at full charge, which would exceed the nRF52840's 3.6 V I/O maximum. No level shifter is needed in the other direction -- I2C is open-drain so no device drives above the pull-up rail, and the MAX17048 reads a 3.3 V bus correctly because its VIH is a fixed 1.4 V (not 0.7*VDD), with SDA/SCL/ALRT rated to +5.5 V absolute max."
+			(at 152.4 88.9 0)
+			(effects
+				(font
+					(size 1.27 1.27)
+				)
+				(hide yes)
+			)
+		)
+		(instances
+			(project "bay-station"
+				(path "/543ba435-6cf4-448c-821e-3c5778b02e9c/615db515-37ad-4c26-9aab-9d4c2fc23c63"
+					(reference "R37")
+					(unit 1)
+				)
+			)
+		)
+	)
+	(symbol
+		(lib_id "Device:R")
+		(at 167.64 88.9 0)
+		(unit 1)
+		(exclude_from_sim no)
+		(in_bom yes)
+		(on_board yes)
+		(dnp no)
+		(property "Reference" "R38"
+			(at 167.64 85.09 0)
+			(effects
+				(font
+					(size 1.27 1.27)
+				)
+			)
+		)
+		(property "Value" "2.2k"
+			(at 167.64 92.71 0)
+			(effects
+				(font
+					(size 1.27 1.27)
+				)
+			)
+		)
+		(property "Footprint" ""
+			(at 167.64 88.9 0)
+			(effects
+				(font
+					(size 1.27 1.27)
+				)
+				(hide yes)
+			)
+		)
+		(property "Datasheet" "~"
+			(at 167.64 88.9 0)
+			(effects
+				(font
+					(size 1.27 1.27)
+				)
+				(hide yes)
+			)
+		)
+		(property "Description" "I2C SCL pull-up for the same bus. Value derived, not defaulted: Rp(min) = (3V3 - VOL)/IOL = (3.3-0.4)/4mA = 725 ohm from the strongest sink on the bus (MAX17048 datasheet 19-6171 Rev 7: VOL 0.4 V at IOL 4 mA). 2.2k sinks 1.32 mA, well inside that, and by the I2C-bus spec (NXP UM10204, tr = 0.8473*Rp*Cb) allows 161 pF of bus capacitance at 400 kHz versus only 75 pF for a default 4.7k -- too tight for a bus that crosses from power_bms to gnss. MUST pull up to +3V3, NEVER to VBATT_PROT: the MAX17048's VDD is the battery rail and reaches 4.2 V at full charge, which would exceed the nRF52840's 3.6 V I/O maximum. No level shifter is needed in the other direction -- I2C is open-drain so no device drives above the pull-up rail, and the MAX17048 reads a 3.3 V bus correctly because its VIH is a fixed 1.4 V (not 0.7*VDD), with SDA/SCL/ALRT rated to +5.5 V absolute max."
+			(at 167.64 88.9 0)
+			(effects
+				(font
+					(size 1.27 1.27)
+				)
+				(hide yes)
+			)
+		)
+		(instances
+			(project "bay-station"
+				(path "/543ba435-6cf4-448c-821e-3c5778b02e9c/615db515-37ad-4c26-9aab-9d4c2fc23c63"
+					(reference "R38")
+					(unit 1)
+				)
+			)
+		)
+	)
+	(symbol
+		(lib_id "Device:R")
+		(at 182.88 88.9 0)
+		(unit 1)
+		(exclude_from_sim no)
+		(in_bom yes)
+		(on_board yes)
+		(dnp no)
+		(property "Reference" "R39"
+			(at 182.88 85.09 0)
+			(effects
+				(font
+					(size 1.27 1.27)
+				)
+			)
+		)
+		(property "Value" "2.2k"
+			(at 182.88 92.71 0)
+			(effects
+				(font
+					(size 1.27 1.27)
+				)
+			)
+		)
+		(property "Footprint" ""
+			(at 182.88 88.9 0)
+			(effects
+				(font
+					(size 1.27 1.27)
+				)
+				(hide yes)
+			)
+		)
+		(property "Datasheet" "~"
+			(at 182.88 88.9 0)
+			(effects
+				(font
+					(size 1.27 1.27)
+				)
+				(hide yes)
+			)
+		)
+		(property "Description" "Pull-up for the MAX17048 ALRT output, which is open-drain and cannot assert a high level on its own (datasheet 19-6171 Rev 7). Value derived, not defaulted: Rp(min) = (3V3 - VOL)/IOL = (3.3-0.4)/4mA = 725 ohm from the strongest sink on the bus (MAX17048 datasheet 19-6171 Rev 7: VOL 0.4 V at IOL 4 mA). 2.2k sinks 1.32 mA, well inside that, and by the I2C-bus spec (NXP UM10204, tr = 0.8473*Rp*Cb) allows 161 pF of bus capacitance at 400 kHz versus only 75 pF for a default 4.7k -- too tight for a bus that crosses from power_bms to gnss. MUST pull up to +3V3, NEVER to VBATT_PROT: the MAX17048's VDD is the battery rail and reaches 4.2 V at full charge, which would exceed the nRF52840's 3.6 V I/O maximum. No level shifter is needed in the other direction -- I2C is open-drain so no device drives above the pull-up rail, and the MAX17048 reads a 3.3 V bus correctly because its VIH is a fixed 1.4 V (not 0.7*VDD), with SDA/SCL/ALRT rated to +5.5 V absolute max."
+			(at 182.88 88.9 0)
+			(effects
+				(font
+					(size 1.27 1.27)
+				)
+				(hide yes)
+			)
+		)
+		(instances
+			(project "bay-station"
+				(path "/543ba435-6cf4-448c-821e-3c5778b02e9c/615db515-37ad-4c26-9aab-9d4c2fc23c63"
+					(reference "R39")
+					(unit 1)
+				)
+			)
 		)
 	)
