File: wristband/programming_debug.kicad_sch (KiCad schematic)
At the start: 1 part, among them J3 Conn_ARM_JTAG_SWD_10

Commit message: Convert global labels to power symbols; import footprints to PCB
Continues the ground cleanup from 0263e7f across the rest of the wristband
sheets: global labels replaced with explicit power symbols and wired
junctions, so connections are drawn rather than implied by name.

                     wires      labels      junctions   symbols
  power_bms          61 -> 83   61 -> 51    0 -> 3      25 -> 36
  programming_debug   7 ->  8    7 ->  4    0 -> 1       1 ->  3
  radio_mcu          71 -> 79   64 -> 42    7 -> 17     18 -> 32
  regulation          7 ->  7    7 ->  4    0 -> 0       3 ->  6

The added symbols are all power ports, so the BOM is untouched: still 47
components, 76 nets, 42 no-connects, 35 analyzer findings with 1 error --
identical before and after. The one error is the known DW01A false
positive (U1.6 GND sits on CELL_N by design, per the reference circuit).

Also ran Update PCB from Schematic on the wristband: 0 -> 46 footprints.
Nothing routed yet, no zones, board outline unchanged.

Co-Authored-By: Claude Opus 5 (1M context) <noreply@anthropic.com>
Changed lines of the file:
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@@
 		)
+	)
+	(junction
+		(at 152.4 123.19)
+		(diameter 0)
+		(color 0 0 0 0)
 	)
 	(no_connect
@@
 	(wire
 		(pts
+			(xy 149.86 116.84) (xy 149.86 123.19)
+		)
+		(stroke
+			(width 0)
+			(type default)
+		)
+	)
+	(wire
+		(pts
+			(xy 149.86 123.19) (xy 152.4 123.19)
+		)
+		(stroke
+			(width 0)
+			(type default)
+		)
+	)
+	(wire
+		(pts
 			(xy 165.1 99.06) (xy 175.26 99.06)
 		)
@@
 	(wire
 		(pts
-			(xy 149.86 116.84) (xy 149.86 127)
-		)
-		(stroke
-			(width 0)
-			(type default)
-		)
-	)
-	(wire
-		(pts
 			(xy 165.1 104.14) (xy 175.26 104.14)
 		)
@@
 	(wire
 		(pts
-			(xy 152.4 86.36) (xy 152.4 76.2)
-		)
-		(stroke
-			(width 0)
-			(type default)
-		)
-	)
-	(wire
-		(pts
-			(xy 152.4 116.84) (xy 152.4 127)
+			(xy 152.4 76.2) (xy 152.4 86.36)
+		)
+		(stroke
+			(width 0)
+			(type default)
+		)
+	)
+	(wire
+		(pts
+			(xy 152.4 116.84) (xy 152.4 123.19)
 		)
 		(stroke
@@
 		)
 	)
-	(global_label "+3V3"
-		(shape input)
-		(at 152.4 76.2 90)
-		(effects
-			(font
-				(size 1.27 1.27)
-			)
-			(justify left)
-		)
-		(property "Intersheetrefs" "${INTERSHEET_REFS}"
-			(at 152.4 76.2 0)
-			(hide yes)
-			(show_name no)
-			(do_not_autoplace no)
-			(effects
-				(font
-					(size 1.27 1.27)
-				)
-			)
-		)
-	)
-	(global_label "GND"
-		(shape input)
-		(at 152.4 127 90)
-		(effects
-			(font
-				(size 1.27 1.27)
-			)
-			(justify left)
-		)
-		(property "Intersheetrefs" "${INTERSHEET_REFS}"
-			(at 152.4 127 0)
-			(hide yes)
-			(show_name no)
-			(do_not_autoplace no)
-			(effects
-				(font
-					(size 1.27 1.27)
-				)
-			)
-		)
-	)
 	(global_label "SWO"
 		(shape input)
@@
 		)
 	)
-	(global_label "GND"
-		(shape input)
-		(at 149.86 127 90)
-		(effects
-			(font
-				(size 1.27 1.27)
-			)
-			(justify left)
-		)
-		(property "Intersheetrefs" "${INTERSHEET_REFS}"
-			(at 149.86 127 0)
-			(hide yes)
-			(show_name no)
-			(do_not_autoplace no)
-			(effects
-				(font
-					(size 1.27 1.27)
-				)
-			)
-		)
-	)
 	(global_label "SWDCLK"
 		(shape input)
@@
 				(font
 					(size 1.27 1.27)
+				)
+			)
+		)
+	)
+	(symbol
+		(lib_id "power:GND")
+		(at 152.4 123.19 0)
+		(unit 1)
+		(body_style 1)
+		(exclude_from_sim no)
+		(in_bom yes)
+		(on_board yes)
+		(in_pos_files yes)
+		(dnp no)
+		(fields_autoplaced yes)
+		(property "Reference" "#PWR021"
+			(at 152.4 129.54 0)
+			(hide yes)
+			(show_name no)
+			(do_not_autoplace no)
+			(effects
+				(font
+					(size 1.27 1.27)
+				)
+			)
+		)
+		(property "Value" "GND"
+			(at 152.4 128.27 0)
+			(show_name no)
+			(do_not_autoplace no)
+			(effects
+				(font
+					(size 1.27 1.27)
+				)
+			)
+		)
+		(property "Footprint" ""
+			(at 152.4 123.19 0)
+			(hide yes)
+			(show_name no)
+			(do_not_autoplace no)
+			(effects
+				(font
+					(size 1.27 1.27)
+				)
+			)
+		)
+		(property "Datasheet" ""
+			(at 152.4 123.19 0)
+			(hide yes)
+			(show_name no)
+			(do_not_autoplace no)
+			(effects
+				(font
+					(size 1.27 1.27)
+				)
+			)
+		)
+		(property "Description" "Power symbol creates a global label with name \"GND\" , ground"
+			(at 152.4 123.19 0)
+			(hide yes)
+			(show_name no)
+			(do_not_autoplace no)
+			(effects
+				(font
+					(size 1.27 1.27)
+				)
+			)
+		)
+		(pin "1"
+		)
+		(instances
+			(project "wristband"
+				(path "/b3417696-fb19-4c3e-bd30-28bb2d157bef/ddd7aa1e-0d16-49f7-8332-00365f7ee71d"
+					(reference "#PWR021")
+					(unit 1)
 				)
 			)
@@
 		(dnp no)
 		(property "Reference" "J3"
-			(at 149.86 118.11 0)
+			(at 139.446 110.49 0)
 			(show_name no)
 			(do_not_autoplace no)
@@
 		)
 		(property "Value" "Conn_ARM_JTAG_SWD_10"
-			(at 149.86 115.57 0)
+			(at 137.922 96.774 0)
 			(show_name no)
 			(do_not_autoplace no)
@@
 					(unit 1)
 				)
+			)
+		)
+	)
+	(symbol
+		(lib_id "power:+3V3")
+		(at 152.4 76.2 0)
+		(unit 1)
+		(body_style 1)
+		(exclude_from_sim no)
+		(in_bom yes)
+		(on_board yes)
+		(in_pos_files yes)
+		(dnp no)
+		(fields_autoplaced yes)
+		(property "Reference" "#PWR022"
+			(at 152.4 80.01 0)
+			(hide yes)
+			(show_name no)
+			(do_not_autoplace no)
+			(effects
+				(font
+					(size 1.27 1.27)
+				)
+			)
+		)
+		(property "Value" "+3V3"
+			(at 152.4 71.12 0)
+			(show_name no)
+			(do_not_autoplace no)
+			(effects
+				(font
+					(size 1.27 1.27)
+				)
+			)
+		)
+		(property "Footprint" ""
+			(at 152.4 76.2 0)
+			(hide yes)
+			(show_name no)
+			(do_not_autoplace no)
+			(effects
+				(font
+					(size 1.27 1.27)
+				)
+			)
+		)
+		(property "Datasheet" ""
+			(at 152.4 76.2 0)
+			(hide yes)
+			(show_name no)
+			(do_not_autoplace no)
+			(effects
+				(font
+					(size 1.27 1.27)
+				)
+			)
+		)
+		(property "Description" "Power symbol creates a global label with name \"+3V3\""
+			(at 152.4 76.2 0)
+			(hide yes)
+			(show_name no)
+			(do_not_autoplace no)
+			(effects
+				(font
+					(size 1.27 1.27)
+				)
+			)
+		)
+		(pin "1"
+		)
+		(instances
+			(project "wristband"
+				(path "/b3417696-fb19-4c3e-bd30-28bb2d157bef/ddd7aa1e-0d16-49f7-8332-00365f7ee71d"
+					(reference "#PWR022")
+					(unit 1)
+				)

Commit message: Migrate wristband to DWM3001C; swap LDO to TPS7A02; fix ERC
Replace the NINA-B400 + DWM3000 pair with a single Qorvo DWM3001C, then
replace the MCP1700 LDO with a nanopower TI TPS7A0233. Wristband ERC goes
from 1 error / 13 warnings to 0 errors / 1 warning.

DWM3001C (U4), verified against Qorvo DS Rev B May 2022:
- Integrates DW3110 UWB + nRF52833 BLE MCU + LIS2DH12 + UWB antenna +
  Bluetooth chip antenna + 38.4MHz crystal. Its nRF52833 is now the host,
  so U3 (NINA-B400) is deleted.
- The DW3110<->nRF52833 SPI is internal, so the board-level UWB SPI bus,
  IRQ/RSTn/WAKEUP, the GPIO5/6 SPI-mode straps (R7/R8), the IRQ pulldown
  (R9) and the external LFXO (Y1/C14/C15) are all gone. C8-C10 too.
- AE1 (PRO-IS-237) removed: the module carries both antennas, so
  antenna.kicad_sch is documentation-only and places nothing.
- SWD moved for the first time: SWD_CLK=2, SWD_DIO=3, RESET=47 (P0.18),
  SWO=28 (P1.00). Battery sense moved to P0.02 = AIN0. Both P1.00=SWO and
  P0.02=AIN0 confirmed in nRF52833 PS v1.7 p825-826.
- Symbol + DWM3001C_PLACEHOLDER footprint are wristband-only, in libs/.
  The footprint has TWO unresolved dimensions (side pitch back-derives to
  1.06375mm; bottom pad row width undimensioned and apparently off-centre).
  VERIFY BEFORE FAB.

TPS7A0233PDBVR (U5), verified against TI SBVS277C:
- Iq 1.6uA typ / 4uA max -> 25nA typ / 46nA max; it was the largest single
  standby draw, bigger than the DWM3001C's own 850nA sleep. Board standby
  ~4.3uA -> ~2.7uA. Accuracy +/-1.5% vs +/-2.5%.
- Not a drop-in: SOT-23-5 1=IN 2=GND 3=EN 4=NC 5=OUT. EN ties to VBAT
  because TPS7A02 is disabled when EN floats and the MCU on this rail
  cannot enable its own supply.
- C12 1uF -> 2.2uF for the 0.5uF effective-capacitance stability floor.
- Symbol is self-contained: KiCad ships no TPS7A02, and every TPS7A05
  sibling is extends-based, which kicad-cli cannot load.

ERC fixes:
- Real bug: regulation.kicad_sch had no labels at all, so U5's input and
  C11 sat on an iso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
Other:
- note added: "SWD / ARM Cortex Debug header for DWM3001C (U4)"
- note added: "SWO=28 (P1.00) -- Qorvo DS Rev B Table 2; P1.00=TRACEDATA[0]/SWO"
- note added: "Standard 2x5 1.27mm pitch. Module-side pin numbers changed with"
- note added: "and AIN mappings confirmed in nRF52833 PS v1.7 p825-826."
- note added: "the DWM3001C migration: SWD_CLK=2, SWD_DIO=3, RESET=47 (P0.18),"
- note removed: "NINA-B111 this board previously used: SWDCLK=11, SWDIO=15,"
- note removed: "RESET_N=19, SWO=8 -- verified against UBX-19049405 R09 Table 6."
- note removed: "SWD / ARM Cortex Debug header for NINA-B400 (U3)"
- note removed: "Standard 2x5 1.27mm pitch. Pin numbers are unchanged from the"
Changed lines of the file:
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@@
 		(comment 1 "Wristband NINA-B400 SWD/debug header -- placement only, not yet wired")
 	)
-	(text "Standard 2x5 1.27mm pitch. Pin numbers are unchanged from the"
+	(text "and AIN mappings confirmed in nRF52833 PS v1.7 p825-826."
+		(exclude_from_sim no)
+		(at 101.6 60.96 0)
+		(effects
+			(font
+				(size 1.7 1.7)
+				(bold yes)
+			)
+			(justify left)
+		)
+	)
+	(text "Standard 2x5 1.27mm pitch. Module-side pin numbers changed with"
 		(exclude_from_sim no)
 		(at 101.6 45.72 0)
@@
 		)
 	)
-	(text "NINA-B111 this board previously used: SWDCLK=11, SWDIO=15,"
+	(text "the DWM3001C migration: SWD_CLK=2, SWD_DIO=3, RESET=47 (P0.18),"
 		(exclude_from_sim no)
 		(at 101.6 50.8 0)
@@
 		)
 	)
-	(text "SWD / ARM Cortex Debug header for NINA-B400 (U3)"
+	(text "SWD / ARM Cortex Debug header for DWM3001C (U4)"
 		(exclude_from_sim no)
 		(at 101.6 40.64 0)
@@
 		)
 	)
-	(text "RESET_N=19, SWO=8 -- verified against UBX-19049405 R09 Table 6."
+	(text "SWO=28 (P1.00) -- Qorvo DS Rev B Table 2; P1.00=TRACEDATA[0]/SWO"
 		(exclude_from_sim no)
 		(at 101.6 55.88 0)
@@
 	(text "VTref takes the regulated +3V3 rail."
 		(exclude_from_sim no)
-		(at 101.6 60.96 0)
+		(at 101.6 66.04 0)
 		(effects
 			(font
@@
 		)
 		(property "Value" "Conn_ARM_JTAG_SWD_10"
-			(at 137.922 96.774 0)
-			(show_name no)
-			(do_not_autoplace no)
+			(at 136.652 93.98 0)
+			(show_name no)
+			(do_not_autoplace no)
