File: wristband/power_bms.kicad_sch (KiCad schematic)
At the start: 18 parts, among them J1 USB4125-GF-A, Q1 AO3401A, Q2 FS8205A, U1 DW01A, U2 MCP73831T-2ACI/OT

Commit message: Land the wristband branch on main: DWM3001C wiring, TPS7A02 LDO, PCB (#5)
Brings six months of `dwm3001c-migration` onto current `main` as one commit.
A true rebase was attempted first and abandoned: the branch's own first
commit is a NINA-B400 migration that commit five then throws away, so
replaying it meant resolving 16 files of conflict for a design state nobody
wants. Squashed to a single three-way merge instead -- 18 conflicts, one
pass.

Both sides had independently migrated the wristband to the DWM3001C, so this
was not a fast-forward. Resolution, by ERC evidence rather than recency:

  main's wristband     104 violations, 93 errors
  branch's wristband     1 violation,   0 errors

main's 93 are 80 pin_not_connected + 10 power_pin_not_driven + 3
pin_not_driven -- PR #1 swapped in a fresh radio sheet and never wired it.
The branch wired it. So the branch's schematics are the base here, not
main's.

Taken from the branch: radio_mcu, regulation, programming_debug,
power_bms, mechanical, libs/, the PCB (9.8k lines, main has none), and the
DWM3001C footprint placeholder.

Taken from main: all project-wide docs. The branch's were stale on the bay
station -- still ESP32-S3 and DWM3000, which main replaced with BT840 and
DW3210.

Reconciled by hand:
- wristband.kicad_sch now carries main's 7-sheet hierarchy. `antenna` is
  dropped (DWM3001C has both antennas on-module); `indicators` and
  `testpoints` are spliced in from main verbatim, UUIDs preserved, so their
  child sheets' instance paths still resolve -- both roots share the root
  UUID b3417696, and the paths check out.
- decisions.md, passives-reference.md and wristband/README.md carried main's
  MCP1700 as the wristband LDO. Rewritten for the TPS7A02, with the swap's
  rationale ported from the branch rather than restated.
- README sheet table corrected: main marked every sheet "Placement only",
  which is no longer true for the five the branch wired.
- Dropped NINA-B400-55_PLACEHOLDER.kicad_mod; that part is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
Parts:
- added D2: Green, LED_SMD:LED_0603_1608Metric, symbol Device:LED
- added D3: ESD5B5.0ST1G, Diode_SMD:D_SOD-523, symbol Device:D_TVS
- added R10: 1k, Resistor_SMD:R_0603_1608Metric, symbol Device:R
- C1, C5: MPN (none) -> CL10B104KB8NNNC; Manufacturer (none) -> Samsung Electro-Mechanics
- C2, C3: MPN (none) -> CL10A475KO8NNNC; Manufacturer (none) -> Samsung Electro-Mechanics
- C4: MPN (none) -> CL10A106KP8NNNC; Manufacturer (none) -> Samsung Electro-Mechanics
- D1: MPN (none) -> ESD5B5.0ST1G; Manufacturer (none) -> onsemi
- J1: MPN (none) -> USB4125-GF-A; Manufacturer (none) -> GCT
- Q1: MPN (none) -> AO3401A; Manufacturer (none) -> Alpha & Omega Semiconductor
- Q2: MPN (none) -> FS8205; Manufacturer (none) -> Fortune Semiconductor
- R1: MPN (none) -> RC0603FR-07100KL; Manufacturer (none) -> Yageo
- R2: MPN (none) -> RC0603FR-13100RL; Manufacturer (none) -> Yageo
- R3: MPN (none) -> RC0603FR-071KL; Manufacturer (none) -> Yageo
- R4: MPN (none) -> RC0603FR-076K8L; Manufacturer (none) -> Yageo
- R5, R6: MPN (none) -> RC0603FR-075K1L; Manufacturer (none) -> Yageo
- U1: MPN (none) -> DW01A; Manufacturer (none) -> Fortune Semiconductor
- U2: MPN (none) -> MCP73831T-2ACI/OT; Manufacturer (none) -> Microchip
Connections:
- net GND: now also J1.SH (SHIELD), D3.2 (A2); no longer J1.S1 (SHIELD)
- net VBUS: now also D3.1 (A1), R10.1
- net CHG_STAT: now reaches U2.1 (STAT)
- net CHG_STAT: now also D2.1 (K)
- new net: D2.2 (A), R10.2
- no-connect marks 1 -> 0
Other:
- note added: "Battery input + reverse-polarity protection"
- note added: "Bulk / bypass on the protected VBAT rail"
- note added: "Cell protection -- DW01A (U1) + FS8205 dual FET (Q2)"
- note added: "Charge status LED -- ~1.3mA via R10 while STAT sinks"
- note added: "Q1 AO3401A as an ideal diode -- no series voltage drop"
- note added: "R5/R6 are the 5.1k CC pull-downs; J1 is power-only (no D+/D-)"
- note added: "U1's GND sits on CELL_N (raw cell -), before the pass FETs,"
- note added: "USB-C charging -- MCP73831, ~147mA set by R4"
- note added: "VBUS ESD -- place close to J1"
- note added: "exactly where Fortune's own application circuit draws it."
- moved on the sheet: BT1, C1, C2, C3, C4, C5, D1, J1, Q1, Q2, R1, R2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
