File: wristband/wristband.kicad_pcb (KiCad board)
At the start: 2 copper layers, 0 parts

Commit message: Land the wristband branch on main: DWM3001C wiring, TPS7A02 LDO, PCB (#5)
Brings six months of `dwm3001c-migration` onto current `main` as one commit.
A true rebase was attempted first and abandoned: the branch's own first
commit is a NINA-B400 migration that commit five then throws away, so
replaying it meant resolving 16 files of conflict for a design state nobody
wants. Squashed to a single three-way merge instead -- 18 conflicts, one
pass.

Both sides had independently migrated the wristband to the DWM3001C, so this
was not a fast-forward. Resolution, by ERC evidence rather than recency:

  main's wristband     104 violations, 93 errors
  branch's wristband     1 violation,   0 errors

main's 93 are 80 pin_not_connected + 10 power_pin_not_driven + 3
pin_not_driven -- PR #1 swapped in a fresh radio sheet and never wired it.
The branch wired it. So the branch's schematics are the base here, not
main's.

Taken from the branch: radio_mcu, regulation, programming_debug,
power_bms, mechanical, libs/, the PCB (9.8k lines, main has none), and the
DWM3001C footprint placeholder.

Taken from main: all project-wide docs. The branch's were stale on the bay
station -- still ESP32-S3 and DWM3000, which main replaced with BT840 and
DW3210.

Reconciled by hand:
- wristband.kicad_sch now carries main's 7-sheet hierarchy. `antenna` is
  dropped (DWM3001C has both antennas on-module); `indicators` and
  `testpoints` are spliced in from main verbatim, UUIDs preserved, so their
  child sheets' instance paths still resolve -- both roots share the root
  UUID b3417696, and the paths check out.
- decisions.md, passives-reference.md and wristband/README.md carried main's
  MCP1700 as the wristband LDO. Rewritten for the TPS7A02, with the swap's
  rationale ported from the branch rather than restated.
- README sheet table corrected: main marked every sheet "Placement only",
  which is no longer true for the five the branch wired.
- Dropped NINA-B400-55_PLACEHOLDER.kicad_mod; that part is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
Parts:
- added BT1: 3.7V LiPo (1S, JST-PH 2-pin), Connector_JST:JST_PH_S2B-PH-K_1x02_P2.00mm_Horizontal, F.Cu at (133.0, 88.5)
- added C1: 0.1uF, Capacitor_SMD:C_0603_1608Metric, F.Cu at (136.0, 85.5)
- added C11: 1uF, Capacitor_SMD:C_0603_1608Metric, F.Cu at (142.5, 81.5)
- added C12: 2.2uF, Capacitor_SMD:C_0603_1608Metric, F.Cu at (142.4, 86.5)
- added C16: 100nF, Capacitor_SMD:C_0603_1608Metric, F.Cu at (117.5, 87.5)
- added C2: 4.7uF, Capacitor_SMD:C_0603_1608Metric, F.Cu at (136.5, 76.5)
- added C3: 4.7uF, Capacitor_SMD:C_0603_1608Metric, F.Cu at (129.7, 87.7)
- added C4: 10uF, Capacitor_SMD:C_0603_1608Metric, F.Cu at (132.7, 84.5)
- added C5: 100nF, Capacitor_SMD:C_0603_1608Metric, F.Cu at (128.5, 92.5)
- added C6: 100nF, Capacitor_SMD:C_0603_1608Metric, F.Cu at (108.5, 74.0)
- added C7: 4.7uF, Capacitor_SMD:C_0603_1608Metric, F.Cu at (108.5, 75.5)
- added D1: ESD5B5.0ST1G, Diode_SMD:D_SOD-523, F.Cu at (110.5, 90.5)
- added D2: Green, LED_SMD:LED_0603_1608Metric, F.Cu at (123.7, 82.0)
- added D3: ESD5B5.0ST1G, Diode_SMD:D_SOD-523, F.Cu at (117.2, 82.0)
- added H1: M2, MountingHole:MountingHole_2.2mm_M2, F.Cu at (141.0, 64.0)
- added H2: M2, MountingHole:MountingHole_2.2mm_M2, F.Cu at (141.5, 91.0)
- added H3: M2, MountingHole:MountingHole_2.2mm_M2, F.Cu at (105.0, 91.0)
- added H4: M2, MountingHole:MountingHole_2.2mm_M2, F.Cu at (104.0, 64.0)
- added J1: USB4125-GF-A, Connector_USB:USB_C_Receptacle_GCT_USB4125-xx-x_6P_TopMnt_Horizontal, F.Cu at (142.0, 74.0)
- added J3: Conn_ARM_JTAG_SWD_10, Connector_PinHeader_1.27mm:PinHeader_2x05_P1.27mm_Vertical, F.Cu at (102.2, 71.0)
- added Q1: AO3401A, Package_TO_SOT_SMD:SOT-23, F.Cu at (127.9, 90.0)
- added Q2: FS8205A, Package_TO_SOT_SMD:SOT-23-6, F.Cu at (138.5, 82.0)
- added R1: 100k, Resistor_SMD:R_0603_1608Metric, F.Cu at (124.0, 89.0)
- added R10: 1k, Resistor_SMD:R_0603_1608Metric, F.Cu at (120.2, 82.0)
- added R11: 1M, Resistor_SMD:R_0603_1608Metric, F.Cu at (113.5, 90.5)
- added R12: 1M, Resistor_SMD:R_0603_1608Metric, F.Cu at (117.5, 90.5)
- added R2: 100, Resistor_SMD:R_0603_1608Metric, F.Cu at (135.3, 83.0)
- added R3: 1k, Resistor_SMD:R_0603_1608Metric, F.Cu at (122.6, 85.5)
- added R4: 6.8k, Resistor_SMD:R_0603_1608Metric, F.Cu at (131.5, 78.0)
- added R5: 5.1k, Resistor_SMD:R_0603_1608Metric, F.Cu at (134.5, 75.5)
- added R6: 5.1k, Resistor_SMD:R_0603_1608Metric, F.Cu at (134.5, 72.3)
- added SW1: SOS, Button_Switch_SMD:Panasonic_EVQPUJ_EVQPUA, F.Cu at (102.0, 82.4)
- added U1: DW01A, Package_TO_SOT_SMD:SOT-23-6, F.Cu at (126.6, 85.5)
- added U2: MCP73831T-2ACI/OT, Package_TO_SOT_SMD:SOT-23-5, F.Cu at (132.1, 81.6)
- added U4: DWM3001C, wristband:DWM3001C_PLACEHOLDER, F.Cu at (120.5, 65.5)
- added U5: TPS7A0233PDBVR, Package_TO_SOT_SMD:SOT-23-5, F.Cu at (142.9, 84.0)
Routing:
- net VBAT_SENSE: track 0.00 -> 5.37 mm
- net +3V3: track 0.00 -> 4.15 mm, vias 0 -> 1
- net PROT_CS: track 0.00 -> 2.04 mm
- net Net-(D2-A): track 0.00 -> 1.89 mm
- net VBAT: track 0.00 -> 1.55 mm, vias 0 -> 1
- net VBUS: track 0.00 -> 1.47 mm
- net GND: vias 0 -> 31
- net CELL_P: vias 0 -> 8
- net CELL_N: vias 0 -> 8
- added copper zone on B.Cu, net CELL_N
- added copper zone on F.Cu, net CELL_N
- added copper zone on In1.Cu, net CELL_N
- added copper zone on In2.Cu, net CELL_N
- added copper zone on B.Cu, net CELL_P
- added copper zone on F.Cu, net CELL_P
- added copper zone on In1.Cu, net CELL_P
- added copper zone on In2.Cu, net CELL_P
Other:
- board outline added: 45 x 35 mm
- copper layers 2 -> 4
- board text added: "Wristband v0 -- 45 x 35 mm, 4-layer. Stackup intent: F.Cu signal / In1.Cu GND plane / In2.Cu power / B.Cu signal. Solid In1.Cu ground reference is required under the DWM3000 UWB and NINA-B400 BLE sections. Outline and size are a STARTING POINT -- confirm against enclosure and strap before layout."
