File: wristband/wristband.kicad_sch (KiCad schematic)
At the start: 0 parts

Commit message: Wristband: consolidate onto one DWM3001C, delete the antenna sheet
The tag's BLE radio turned out to serve no purpose -- it talks only over
UWB. Once BLE is not a requirement the question stops being "which BLE
module" and becomes "what is the simplest way to get a Cortex-M4 talking to
a DW3110". That is one DWM3001C: DW3110 transceiver, nRF52833 MCU, LIS2DH12
accelerometer, both antennas, power management and crystal in one part.

Counterintuitively this is the simpler board. A discrete MCU would have
added a second part plus its crystal, decoupling, layout and an inter-chip
SPI bus.

Removed: NINA-B111, DWM3000, antenna.kicad_sch in full (ProAnt InSide-2400,
U.FL connector, L/C matching network), R7/R8 GPIO5/6 straps and R9 IRQ
pulldown -- the host-to-transceiver link is internal now. 8 sheets to 6.
Also closes the "matching-network values pending RF tuning" open item;
there is nothing left to tune.

BLE and the accelerometer are deliberately unused -- dormant silicon on a
module bought for its M4 and its UWB radio. The accelerometer is worth
revisiting to motion-gate the UWB, the largest battery lever available on
the power-constrained side of the system.

Symbol hand-authored, all 48 pins from the real Qorvo DWM3001C Data Sheet
Rev B (May 2022) Table 2, via pdftotext -raw. Caveat carried in the symbol:
pin 18 is not documented in that table, so it is modelled as a passive NC.
Footprint should be imported from a vendor library, not hand-authored --
the land pattern is Figure 5, a drawing.

Side effect: shared/ now contains nothing either board uses. The DWM3000
symbol is kept there deliberately as the fallback until the bay station's
discrete rework is proven.

LDO budget got easier, not harder: 70 mA to 43 mA, headroom 3.6x to 5.8x.
One module doing both jobs draws less than two doing one each.

Also corrects the original DWM3001C rejection in shared/README.md, which
compared it against DWM3000 while holding NINA-B111 fixed -- it never
evaluated replacing both.
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
Other:
- removed sheet Antenna
- added sheet Indicators (indicators.kicad_sch)
- added sheet Test Points (testpoints.kicad_sch)
Changed lines of the file:
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@@
-	)
-	(sheet
-		(at 210 30)
-		(size 60 40)
-		(fields_autoplaced yes)
-		(stroke
-			(width 0.1524)
-			(type solid)
-		)
-		(fill
-			(color 0 0 0 0.0000)
-		)
-		(property "Sheetname" "Antenna"
-			(at 210 28.5 0)
-			(effects
-				(font
-					(size 1.27 1.27)
-				)
-				(justify left bottom)
-			)
-		)
-		(property "Sheetfile" "antenna.kicad_sch"
-			(at 210 71.5 0)
-			(effects
-				(font
-					(size 1.27 1.27)
-				)
-				(justify left top)
-			)
-		)
-		(instances
-			(project "wristband"
-				(path "/b3417696-fb19-4c3e-bd30-28bb2d157bef"
-					(page "6")
-				)
-			)
-		)
 	)
 	(sheet
@@
 			(effects
 				(font
+					(size 1.27 1.27)
+				)
+				(justify left top)
+			)
+		)
+		(instances
+			(project "wristband"
+				(path "/b3417696-fb19-4c3e-bd30-28bb2d157bef"
+					(page "7")
+				)
+			)
+		)
+	)
+	(sheet
+		(at 30 170)
+		(size 60 40)
+		(fields_autoplaced yes)
+		(stroke
+			(width 0.1524)
+			(type solid)
+		)
+		(fill
+			(color 0 0 0 0.0000)
+		)
+		(property "Sheetname" "Indicators"
+			(at 30 168.5 0)
+			(effects
+				(font
+					(size 1.27 1.27)
+				)
+				(justify left bottom)
+			)
+		)
+		(property "Sheetfile" "indicators.kicad_sch"
+			(at 30 211.5 0)
+			(effects
+				(font
+					(size 1.27 1.27)
+				)
+				(justify left top)
+			)
+		)
+		(instances
+			(project "wristband"
+				(path "/b3417696-fb19-4c3e-bd30-28bb2d157bef"
+					(page "8")
+				)
+			)
+		)
+	)
+	(sheet
+		(at 210 30)
+		(size 60 40)
+		(fields_autoplaced yes)
+		(stroke
+			(width 0.1524)
+			(type solid)
+		)
+		(fill
+			(color 0 0 0 0.0000)
+		)
+		(property "Sheetname" "Test Points"
+			(at 210 28.5 0)
+			(effects
+				(font
+					(size 1.27 1.27)
+				)
+				(justify left bottom)
+			)
+		)
+		(property "Sheetfile" "testpoints.kicad_sch"
+			(at 210 71.5 0)
+			(effects
+				(font
